Commit message: adjusting so sim works in example workspace

File: veg_bot/worlds_and_models/kuka/kr6r900sixx_macro.xacro (robot description, xacro)
@@ -3,5 +3,5 @@
   <xacro:include filename="$(find veg_bot)/worlds_and_models/kuka/common_constants.xacro"/>
   <xacro:include filename="$(find veg_bot)/worlds_and_models/kuka/common_materials.xacro"/>
-  <xacro:include filename="$(find start_creating_robots)/worlds_and_models/krytn/inertial.xacro" />
+  <xacro:include filename="$(find krytn)/robot_description/magni/inertial.xacro" />
   <xacro:macro name="link_weight">
     <xacro:sphere_inertial radius="1" mass="2" />

File: veg_bot/worlds_and_models/kuka/realsense.urdf.xacro (robot description, xacro)
@@ -11,5 +11,5 @@
             <origin xyz="0 0 0" rpy="0 0 1.57"/>
             <geometry>
-                <mesh filename="file://$(find start_creating_robots)/worlds_and_models/krytn/meshes/realsense.dae">
+                <mesh filename="file://$(find veg_bot)/worlds_and_models/kuka/meshes/realsense.dae">
                     <submesh>
                         <name>RealSense</name>
